File: eagle/TreeShield.sch (EAGLE design)
At the start: 65 parts

Commit message: schematic sort of done
Parts:
- removed JP1, JP2, JP3, JP4, JP5: (no value), adafruit:PINHD-1X8BIG
- removed R$0, R$1, R$10, R$11, R$12, R$13, R$14, R$15, R$16, R$17, R$18, R$19, R$2, R$20, R$21, R$22, R$23, R$24, R$25, R$26, R$27, R$28, R$29, R$3, R$30, R$31, R$32, R$33, R$34, R$35, R$36, R$37, R$38, R$39, R$4, R$5, R$6, R$7, R$8, R$9: (no value), resistor:R-US_0817/7V
- removed U$5: CD74ACT164M, elecanisms:CD74ACT164M
- added IC1: LM1117T-5.0, lm1117:LM1117T-5.0
- added IC2: 74HC164D, CD74ACT164M:74HC164D
- added R1, R10, R11, R12, R13, R14, R15, R16, R17, R18, R19, R2, R20, R21, R22, R23, R24, R25, R26, R27, R28, R29, R3, R30, R31, R32, R33, R34, R35, R36, R37, R38, R39, R4, R40, R5, R6, R7, R8, R9: (no value), SparkFun-Resistors:RESISTOR0603
- added STAGE12GND, STAGE12PWR, STAGE34GND, STAGE34PWR, STAGE56GND, STAGE56PWR, STAGE78GND, STAGE78PWR: PINHD-1X10, adafruit:PINHD-1X10
- added U1: ARDUINOR3-BPLACE, adafruit:ARDUINOR3-BPLACE
Connections:
- new net N$76: STAGE12GND.1, STAGE12GND.10, STAGE12GND.2, STAGE12GND.3, STAGE12GND.4, STAGE12GND.5, STAGE12GND.6, STAGE12GND.7, STAGE12GND.8, STAGE12GND.9
- net GND: now also IC1.GND, STAGE34GND.1, STAGE34GND.10, STAGE34GND.2, STAGE34GND.3, STAGE34GND.4, STAGE34GND.5, STAGE34GND.6, STAGE34GND.7, STAGE34GND.8, STAGE34GND.9, STAGE56GND.1, STAGE56GND.10, STAGE56GND.2, STAGE56GND.3, STAGE56GND.4, STAGE56GND.5, STAGE56GND.6, STAGE56GND.7, STAGE56GND.8, STAGE56GND.9, STAGE78GND.1, STAGE78GND.10, STAGE78GND.2, STAGE78GND.3, STAGE78GND.4, STAGE78GND.5, STAGE78GND.6, STAGE78GND.7, STAGE78GND.8, STAGE78GND.9, U$1.D1, U$1.D2, U$2.D1, U$2.D2, U$3.D1, U$3.D2, U$4.D1, U$4.D2; no longer U$5.GND
- net N$2: now also D8D13.1, IC2A.A; no longer U$2.D1, U$5.Q0
- net N$20: now also R3.2, STAGE12PWR.3; no longer R$10.1, R$11.1, R$13.1, R$14.1, U$2.G1
- net N$21: now also R4.2, STAGE12PWR.4; no longer R$15.1, R$16.1, R$17.1, R$18.1, R$19.1, U$2.G2
- net N$22: now also R5.2, STAGE12PWR.5; no longer R$20.1, R$21.1, R$23.1, R$24.1, U$4.G1
- net N$23: now also R6.2, STAGE12PWR.6; no longer R$25.1, R$26.1, R$27.1, R$28.1, R$29.1, U$4.G2
- net N$24: now also R7.2, STAGE12PWR.7; no longer R$30.1, R$31.1, R$33.1, R$34.1, U$3.G1
- net N$25: now also R8.2, STAGE12PWR.8; no longer R$35.1, R$36.1, R$37.1, R$38.1, R$39.1, U$3.G2
- net N$26: now also D8D13.3, IC2A.CLK; no longer U$1.D1, U$5.Q2
- net N$27: now also D8D13.4, IC2A.CLR; no longer U$1.D2, U$5.Q3
- net N$28: now also IC2A.QA, U$2.G1; no longer U$4.D1, U$5.Q4
- net N$29: now also IC2A.QB, U$2.G2; no longer U$4.D2, U$5.Q5
- net N$3: now also D8D13.2, IC2A.B; no longer U$2.D2, U$5.Q1
- net N$30: now also IC2A.QC, U$1.G1; no longer U$3.D1, U$5.Q6
- net N$31: now also IC2A.QD, U$1.G2; no longer U$3.D2, U$5.Q7
- net N$32: now also R9.2, STAGE12PWR.9; no longer JP1.1, R$10.2
- net N$33: now also R10.2, STAGE12PWR.10; no longer JP1.2, R$11.2
- net N$34: now also R1.1, R2.1, R3.1, R4.1, R5.1, U$2.S1; no longer JP1.3, R$12.2
- net N$35: now also R10.1, R6.1, R7.1, R8.1, R9.1, U$2.S2; no longer JP1.4, R$13.2
- net N$36: now also R11.2, STAGE34PWR.1; no longer JP1.5, R$14.2
- net N$37: now also R12.2, STAGE34PWR.2; no longer JP1.6, R$15.2
- net N$38: now also R13.2, STAGE34PWR.3; no longer JP1.7, R$16.2
- net N$39: now also R14.2, STAGE34PWR.4; no longer JP1.8, R$17.2
- net N$40: now also R15.2, STAGE34PWR.5; no longer JP2.1, R$18.2
- net N$41: now also R16.2, STAGE34PWR.6; no longer JP2.2, R$19.2
- net N$42: now also R17.2, STAGE34PWR.7; no longer JP2.3, R$0.2
- net N$43: now also R18.2, STAGE34PWR.8; no longer JP2.4, R$1.2
- net N$44: now also R19.2, STAGE34PWR.9; no longer JP2.5, R$2.2
- net N$45: now also R20.2, STAGE34PWR.10; no longer JP2.6, R$3.2
- net N$46: now also R21.2, STAGE56PWR.1; no longer JP2.7, R$4.2
- net N$47: now also R22.2, STAGE56PWR.2; no longer JP2.8, R$5.2
- net N$48: now also R23.2, STAGE56PWR.3; no longer JP3.1, R$6.2
- net N$49: now also R24.2, STAGE56PWR.4; no longer JP3.2, R$7.2
- net N$50: now also R25.2, STAGE56PWR.5; no longer JP3.3, R$8.2
- net N$51: now also R26.2, STAGE56PWR.6; no longer JP3.4, R$9.2
- net N$52: now also R27.2, STAGE56PWR.7; no longer JP3.5, R$20.2
- net N$53: now also R28.2, STAGE56PWR.8; no longer JP3.6, R$21.2
- net N$54: now also R29.2, STAGE56PWR.9; no longer JP3.7, R$22.2
- net N$55: now also R30.2, STAGE56PWR.10; no longer JP3.8, R$23.2
- net N$56: now also R31.2, STAGE78PWR.1; no longer JP4.1, R$24.2
- net N$57: now also R32.2, STAGE78PWR.2; no longer JP4.2, R$25.2
- net N$58: now also R33.2, STAGE78PWR.3; no longer JP4.3, R$26.2
- net N$59: now also R34.2, STAGE78PWR.4; no longer JP4.4, R$27.2
- net N$60: now also R35.2, STAGE78PWR.5; no longer JP4.5, R$28.2
- net N$61: now also R36.2, STAGE78PWR.6; no longer JP4.6, R$29.2
- net N$62: now also R37.2, STAGE78PWR.7; no longer JP4.7, R$30.2
- net N$63: now also R38.2, STAGE78PWR.8; no longer JP4.8
- net N$64: now also R39.2, STAGE78PWR.9; no longer JP5.1, R$32.2
- net N$65: now also R40.2, STAGE78PWR.10; no longer JP5.2, R$33.2
- net N$66: now also R11.1, R12.1, R13.1, R14.1, R15.1, U$1.S1; no longer JP5.3, R$34.2
- net N$67: now also IC2A.QH, U$3.G2; no longer JP5.4, R$35.2
- net N$68: now also IC2A.QG, U$3.G1; no longer JP5.5, R$36.2
- net N$69: now also IC2A.QF, U$4.G2; no longer JP5.6, R$37.2
- net N$70: now also IC2A.QE, U$4.G1; no longer JP5.7, R$38.2
- net N$71: now also R16.1, R17.1, R18.1, R19.1, R20.1, U$1.S2; no longer JP5.8, R$39.2
- net N$72: now also R21.1, R22.1, R23.1, R24.1, R25.1, U$4.S1; no longer D8D13.1, U$5.DS2
- net N$73: now also R26.1, R27.1, R28.1, R29.1, R30.1, U$4.S2; no longer D8D13.2, U$5.DS1
- net N$74: now also R31.1, R32.1, R33.1, R34.1, R35.1, U$3.S1; no longer D8D13.3, U$5.MR'
- net N$75: now also R36.1, R37.1, R38.1, R39.1, R40.1, U$3.S2; no longer D8D13.4, U$5.CP
- net N$8: now also R1.2, STAGE12PWR.1; no longer R$0.1, R$1.1, R$3.1, R$4.1, U$1.G1
- net N$9: now also R2.2, STAGE12PWR.2; no longer R$5.1, R$6.1, R$7.1, R$8.1, R$9.1, U$1.G2
- net VCC: now also IC1.OUT; no longer U$1.S1, U$1.S2, U$2.S1, U$2.S2, U$3.S1, U$3.S2, U$4.S1, U$4.S2, U$5.VCC
- net VDD: now also IC1.IN
Other:
- moved on the sheet: D8D13, U$1, U$4
